File: Hardware/FabAccess.kicad_pcb (KiCad board)
At the start: 2 copper layers, 69.3 x 69 mm, 25 parts, among them J1 FTDI, J2 USB_computer, J3 USB_machine, J4 RFID-RC522, Q1 UMH3N, Q2 MOSFET_N-CH_30V_1.7A, Q3 MOSFET_N-CH_30V_1.7A, SW1 BUTTON_B3SN, U1 LM1117-3.3, U4 ESP-12E

Commit message: KiCAD project
Parts:
- removed J1: FTDI, Connector_PinHeader_2.54mm:PinHeader_2x03_P2.54mm_Vertical_SMD
- removed Q1: UMH3N, Package_TO_SOT_SMD:SOT-363_SC-70-6_Handsoldering
- added FTDI: Conn_01x04, Connector_PinHeader_2.54mm:PinHeader_1x04_P2.54mm_Horizontal, F.Cu at (76.4, 36.4)
- added UPLOAD: BUTTON_B3SN, fab:Button_Omron_B3SN_6x6mm, F.Cu at (85.0, 46.7)
- moved R9 9.45 mm to (77.9, 40.6), turned to 270 degrees
- moved R7 6.50 mm to (75.3, 40.6), turned to 270 degrees
- moved R10 1.55 mm to (75.4, 53.6), turned to 270 degrees
- renumbered SW1 to RESET
Routing:
- net RESET: track 89.5 -> 31.5 mm
- net +3V3: track 101.2 -> 78.8 mm, vias 3 -> 1
- net DTR: track 16.7 -> 0.00 mm, vias 2 -> 0
- net GND: track 221.7 -> 236.4 mm, vias 6 -> 4
- net RTS: track 8.60 -> 0.00 mm
- net Net-(R9-Pad2): track 3.75 -> 12.2 mm
- net IO0: track 18.6 -> 27.0 mm, vias 0 -> 2
- net TX: track 19.1 -> 12.0 mm
- net RX: track 20.9 -> 13.7 mm
Other:
- board text added: "3V3"
- board text removed: "+3.3V"
- board text removed: "DTR"
